File: hw/left_revision3_1.brd (EAGLE design)
At the start: 99.7 x 80.6 mm, 51 parts, among them J2 CAN, U2 MCP2551, X1 7A-20.000MAAJ-T

Commit message: version 3.0 hardware drawn
Parts:
- SW1, SW10, SW11, SW12, SW13, SW14, SW15, SW2, SW3, SW4, SW5, SW6, SW7, SW8, SW9: device usevolt:SWITCH_EVQ9P6B40 -> usevolt:SWITCH_KMR231
Connections:
- net GND: now also SW1.P$2, SW1.P$4, SW10.P$2, SW10.P$4, SW11.P$2, SW11.P$4, SW12.P$2, SW12.P$4, SW13.P$2, SW13.P$4, SW14.P$2, SW14.P$4, SW15.P$2, SW15.P$4, SW2.P$2, SW2.P$4, SW3.P$2, SW3.P$4, SW4.P$2, SW4.P$4, SW5.P$2, SW5.P$4, SW6.P$2, SW6.P$4, SW7.P$2, SW7.P$4, SW8.P$2, SW8.P$4, SW9.P$2, SW9.P$4; no longer SW1.B, SW1.B', SW10.B, SW10.B', SW11.B, SW11.B', SW12.B, SW12.B', SW13.B, SW13.B', SW14.B, SW14.B', SW15.B, SW15.B', SW2.B, SW2.B', SW3.B, SW3.B', SW4.B, SW4.B', SW5.B, SW5.B', SW6.B, SW6.B', SW7.B, SW7.B', SW8.B, SW8.B', SW9.B, SW9.B'
- net SW1: now also SW1.P$1, SW1.P$3; no longer SW1.A, SW1.A'
- net SW10: now also SW10.P$1, SW10.P$3; no longer SW10.A, SW10.A'
- net SW11: now also SW11.P$1, SW11.P$3; no longer SW11.A, SW11.A'
- net SW12: now also SW12.P$1, SW12.P$3; no longer SW12.A, SW12.A'
- net SW13: now also SW13.P$1, SW13.P$3; no longer SW13.A, SW13.A'
- net SW14: now also SW14.P$1, SW14.P$3; no longer SW14.A, SW14.A'
- net SW15: now also SW15.P$1, SW15.P$3; no longer SW15.A, SW15.A'
- net SW2: now also SW2.P$1, SW2.P$3; no longer SW2.A, SW2.A'
- net SW3: now also SW3.P$1, SW3.P$3; no longer SW3.A, SW3.A'
- net SW4: now also SW4.P$1, SW4.P$3; no longer SW4.A, SW4.A'
- net SW5: now also SW5.P$1, SW5.P$3; no longer SW5.A, SW5.A'
- net SW6: now also SW6.P$1, SW6.P$3; no longer SW6.A, SW6.A'
- net SW7: now also SW7.P$1, SW7.P$3; no longer SW7.A, SW7.A'
- net SW8: now also SW8.P$1, SW8.P$3; no longer SW8.A, SW8.A'
- net SW9: now also SW9.P$1, SW9.P$3; no longer SW9.A, SW9.A'
Routing:
- net SW15: track 52.7 -> 49.8 mm
- net TXD: track 32.6 -> 35.2 mm
- net SW11: track 53.6 -> 56.0 mm
- net SW12: track 39.2 -> 36.9 mm
- net SW13: track 31.5 -> 30.0 mm
- net SW4: track 17.4 -> 16.2 mm
- net SW5: track 33.8 -> 32.7 mm
- net SW8: track 11.9 -> 12.7 mm
- net SW7: track 24.7 -> 24.1 mm
- net SW3: track 7.47 -> 8.02 mm
- net SW10: track 38.4 -> 38.9 mm
- net GND: vias 162 -> 176
Other:
- board text added: "Usewood CAN keypad driver Left Rev 3.1"
- board text removed: "Usewood CAN keypad driver Left Rev 3.0"
