File: hw/right_revision3_1.sch (EAGLE design)
At the start: 51 parts, among them J2 CAN, U2 MCP2551, X1 7A-20.000MAAJ-T

Commit message: version 3.0 hardware drawn
Parts:
- SW1, SW10, SW11, SW12, SW13, SW14, SW15, SW2, SW3, SW4, SW5, SW6, SW7, SW8, SW9: device usevolt:SWITCH_EVQP6L -> usevolt:SWITCH_KMR231G
Changed lines of the file:
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@@
 <part name="C19" library="usevolt" deviceset="CAP" device="_0603" value="100n"/>
 <part name="J1" library="usevolt" deviceset="HEADER_USART_2" device="_SMD"/>
-<part name="SW11" library="usevolt" deviceset="SWITCH_EVQP6L" device=""/>
-<part name="SW12" library="usevolt" deviceset="SWITCH_EVQP6L" device=""/>
-<part name="SW6" library="usevolt" deviceset="SWITCH_EVQP6L" device=""/>
-<part name="SW7" library="usevolt" deviceset="SWITCH_EVQP6L" device=""/>
-<part name="SW8" library="usevolt" deviceset="SWITCH_EVQP6L" device=""/>
-<part name="SW13" library="usevolt" deviceset="SWITCH_EVQP6L" device=""/>
-<part name="SW14" library="usevolt" deviceset="SWITCH_EVQP6L" device=""/>
-<part name="SW9" library="usevolt" deviceset="SWITCH_EVQP6L" device=""/>
+<part name="SW11" library="usevolt" deviceset="SWITCH_KMR231G" device=""/>
+<part name="SW12" library="usevolt" deviceset="SWITCH_KMR231G" device=""/>
+<part name="SW6" library="usevolt" deviceset="SWITCH_KMR231G" device=""/>
+<part name="SW7" library="usevolt" deviceset="SWITCH_KMR231G" device=""/>
+<part name="SW8" library="usevolt" deviceset="SWITCH_KMR231G" device=""/>
+<part name="SW13" library="usevolt" deviceset="SWITCH_KMR231G" device=""/>
+<part name="SW14" library="usevolt" deviceset="SWITCH_KMR231G" device=""/>
+<part name="SW9" library="usevolt" deviceset="SWITCH_KMR231G" device=""/>
 <part name="GND7" library="supply1" deviceset="GND" device=""/>
-<part name="SW4" library="usevolt" deviceset="SWITCH_EVQP6L" device=""/>
-<part name="SW5" library="usevolt" deviceset="SWITCH_EVQP6L" device=""/>
-<part name="SW3" library="usevolt" deviceset="SWITCH_EVQP6L" device=""/>
-<part name="SW2" library="usevolt" deviceset="SWITCH_EVQP6L" device=""/>
-<part name="SW1" library="usevolt" deviceset="SWITCH_EVQP6L" device=""/>
-<part name="SW15" library="usevolt" deviceset="SWITCH_EVQP6L" device=""/>
-<part name="SW10" library="usevolt" deviceset="SWITCH_EVQP6L" device=""/>
+<part name="SW4" library="usevolt" deviceset="SWITCH_KMR231G" device=""/>
+<part name="SW5" library="usevolt" deviceset="SWITCH_KMR231G" device=""/>
+<part name="SW3" library="usevolt" deviceset="SWITCH_KMR231G" device=""/>
+<part name="SW2" library="usevolt" deviceset="SWITCH_KMR231G" device=""/>
+<part name="SW1" library="usevolt" deviceset="SWITCH_KMR231G" device=""/>
+<part name="SW15" library="usevolt" deviceset="SWITCH_KMR231G" device=""/>
+<part name="SW10" library="usevolt" deviceset="SWITCH_KMR231G" device=""/>
 </parts>
 <sheets>
