File: hw/left.brd (EAGLE design)
At the start: 99.7 x 80.6 mm, 51 parts, among them J2 CAN, U2 MCP2551, X1 7A-20.000MAAJ-T

Commit message: developing HW version 4.0
Parts:
- removed D16, D17, D18: PDZ3.3B,115, usevolt:SOD123
- removed J1: (no value), usevolt:HEADER_4_2_SMD
- added D4, D5, D6: (no value), usevolt:DO219AB
- C18, C2: value EEE1JA101P -> 100uF; device usevolt:CAP_POL_SMD_10X10X10MM -> usevolt:CAP_POL_8.3X8.3MM
- D1: device arm:DO-214AB -> usevolt:DO-214AA
- SW1, SW10, SW11, SW12, SW13, SW14, SW15, SW2, SW3, SW4, SW5, SW6, SW7, SW8, SW9: device usevolt:SWITCH_KMR231 -> usevolt:SWITCH_KSC421J-70SH-LFS
- U$1: device usevolt:MOLEX_MICRO_FIT_10WAY_SMD -> usevolt:MOLEX_MICRO-FIT_10WAY_V
- moved D1 65.9 mm to (84.7, 73.3), flipped to the top
- moved C16 64.1 mm to (89.2, 80.3), flipped to the top
- moved C18 64.1 mm to (68.7, 65.4), flipped to the top
- moved C19 64.1 mm to (87.4, 80.3), flipped to the top
- moved D2 64.1 mm to (62.5, 70.5), flipped to the top
- moved D3 64.1 mm to (97.5, 82.7), flipped to the top
- moved F1 64.1 mm to (92.2, 73.6), flipped to the top
- moved L1 64.1 mm to (80.5, 64.2), flipped to the top
- moved R21 64.1 mm to (97.5, 86.2), flipped to the top
- moved R22 64.1 mm to (60.7, 70.5), flipped to the top
- moved VR1 64.1 mm to (72.6, 69.9), flipped to the top
- moved VR2 64.1 mm to (67.4, 69.2), flipped to the top
- moved C1 64.1 mm to (73.3, 75.3), flipped to the top
- moved C17 64.1 mm to (77.4, 70.5), flipped to the top
- moved C7 64.1 mm to (64.3, 70.5), flipped to the top
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Connections:
- net +3V3: now also D4.P$2, D5.P$2, D6.P$2
- net +5V: now also C18.P$2; no longer C18.+, J1.P$4, J1.P$5
- net AD0: now also D4.P$1; no longer D18.P$2
- net AD1: now also D6.P$1; no longer D16.P$2
- net AD2: now also D5.P$1; no longer D17.P$2
- net GND: now also C18.P$1, C2.P$1, SW1.P$3, SW10.P$3, SW11.P$3, SW12.P$3, SW13.P$3, SW14.P$3, SW15.P$3, SW2.P$3, SW3.P$3, SW4.P$3, SW5.P$3, SW6.P$3, SW7.P$3, SW8.P$3, SW9.P$3; no longer C18.-, C2.-, D16.P$1, D17.P$1, D18.P$1, J1.P$2, J1.P$7, SW1.P$2, SW10.P$2, SW11.P$2, SW12.P$2, SW13.P$2, SW14.P$2, SW15.P$2, SW2.P$2, SW3.P$2, SW4.P$2, SW5.P$2, SW6.P$2, SW7.P$2, SW8.P$2, SW9.P$2
- net N$4: now also C2.P$2; no longer C2.+
- net RXD: no longer J1.P$3, J1.P$6
- net SW1: now also SW1.P$2; no longer SW1.P$3
- net SW10: now also SW10.P$2; no longer SW10.P$3
- net SW11: now also SW11.P$2; no longer SW11.P$3
- net SW12: now also SW12.P$2; no longer SW12.P$3
- net SW13: now also SW13.P$2; no longer SW13.P$3
- net SW14: now also SW14.P$2; no longer SW14.P$3
- net SW15: now also SW15.P$2; no longer SW15.P$3
- net SW2: now also SW2.P$2; no longer SW2.P$3
- net SW3: now also SW3.P$2; no longer SW3.P$3
- net SW4: now also SW4.P$2; no longer SW4.P$3
- net SW5: now also SW5.P$2; no longer SW5.P$3
- net SW6: now also SW6.P$2; no longer SW6.P$3
- net SW7: now also SW7.P$2; no longer SW7.P$3
- net SW8: now also SW8.P$2; no longer SW8.P$3
- net SW9: now also SW9.P$2; no longer SW9.P$3
- net TXD: no longer J1.P$1, J1.P$8
Routing:
- net SW11: track 56.0 -> 0.00 mm, vias 1 -> 0
- net AD2: track 53.3 -> 0.00 mm
- net SW15: track 49.8 -> 0.00 mm, vias 1 -> 0
- net AD1: track 46.1 -> 0.00 mm
- net SW6: track 42.1 -> 0.00 mm, vias 1 -> 0
- net AD0: track 41.3 -> 0.00 mm
- net SW1: track 39.7 -> 0.00 mm, vias 1 -> 0
- net GND: track 39.6 -> 0.00 mm, vias 176 -> 0
- net SW10: track 38.9 -> 0.00 mm, vias 1 -> 0
- net SW12: track 36.9 -> 0.00 mm, vias 1 -> 0
- net TXD: track 35.2 -> 0.00 mm, vias 2 -> 0
- net SW14: track 34.5 -> 0.00 mm, vias 1 -> 0
- net SW5: track 32.7 -> 0.00 mm, vias 1 -> 0
- net SW13: track 30.0 -> 0.00 mm, vias 1 -> 0
- net RXD: track 24.8 -> 0.00 mm
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- removed copper zone on layer 16, net +3V3
- removed copper zone on layer 16, net +5V
- removed copper zone on layer 16, net N$11
- removed copper zone on layer 16, net N$32
- removed copper zone on layer 16, net N$4
- removed copper zone on layer 16, net VDD
Other:
- board text added: "Usewood CAN keypad driver Left Rev 4"
- board text removed: "Usewood CAN keypad driver Left Rev 3.1"
