File: hw/left.sch (EAGLE design)
At the start: 51 parts, among them J2 CAN, U2 MCP2551, X1 7A-20.000MAAJ-T

Commit message: developing HW version 4.0
Parts:
- removed D16, D17, D18: PDZ3.3B,115, usevolt:DIODE_ZENERSDO123
- removed J1: (no value), usevolt:HEADER_USART_2_SMD
- added D4, D5, D6: (no value), usevolt:DIODEDO219AB
- C18, C2: value EEE1JA101P -> 100uF; device usevolt:CAP_POLSMD_10X10X10MM -> usevolt:CAP_EEE-FK1H470P
- D1: device arm:DIODE_TVSDO-214AA -> usevolt:DIODE_TVS_SMBJ33A-TRDO-214AA
- SW1, SW10, SW11, SW12, SW13, SW14, SW15, SW2, SW3, SW4, SW5, SW6, SW7, SW8, SW9: device usevolt:SWITCH_KMR231G -> usevolt:SWITCH_KSC421J-70SH-LFS
- U$1: device usevolt:MOLEX_MICRO-FIT_10WAY_SMD -> usevolt:MOLEX_MICRO-FIT_10WAY_V
Connections:
- net +3V3: now also D4.N, D5.N, D6.N
- net +5V: no longer J1.+5V, J1.+5V@1
- net AD0: now also D4.P; no longer D18.N
- net AD1: now also D6.P; no longer D16.N
- net AD2: now also D5.P; no longer D17.N
- net GND: no longer D16.P, D17.P, D18.P, J1.GND, J1.GND@1
- net RXD: no longer J1.TX, J1.TX@1
- net TXD: no longer J1.RX, J1.RX@1
Other:
- note added: "Revision 4.0"
- note added: "Usewood keypad (c) Usevolt Oy"
- note removed: "Release updates:"
- note removed: "Usewood keypad CAN driver"
- moved on the sheet: U$1
