File: hw/right.brd (EAGLE design)
At the start: 99.7 x 80.6 mm, 51 parts, among them J2 CAN, U2 MCP2551, X1 7A-20.000MAAJ-T

Commit message: developing HW version 4.0
Parts:
- C18, C2: value EEE1JA101P -> 100uF
- U$1: device usevolt:MOLEX_MICRO_FIT_10WAY_SMD -> usevolt:MOLEX-MICRO-FIT_10WAY
Routing:
- net SW11: track 55.0 -> 0.00 mm, vias 1 -> 0
- net SW15: track 49.3 -> 0.00 mm, vias 1 -> 0
- net SW6: track 42.9 -> 0.00 mm, vias 1 -> 0
- net AD0: track 42.4 -> 0.00 mm
- net SW1: track 41.1 -> 0.00 mm, vias 1 -> 0
- net AD1: track 38.8 -> 0.00 mm
- net SW10: track 38.4 -> 0.00 mm, vias 1 -> 0
- net SW12: track 36.1 -> 0.00 mm, vias 1 -> 0
- net SW5: track 34.1 -> 0.00 mm, vias 1 -> 0
- net SW14: track 31.9 -> 0.00 mm, vias 1 -> 0
- net AD2: track 31.7 -> 0.00 mm
- net SW13: track 27.5 -> 0.00 mm, vias 1 -> 0
- net SW7: track 23.5 -> 0.00 mm, vias 1 -> 0
- net SW2: track 21.2 -> 0.00 mm, vias 1 -> 0
- net SW9: track 19.3 -> 0.00 mm, vias 1 -> 0
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- removed copper zone on layer 16, net +5V
- removed copper zone on layer 16, net N$11
- removed copper zone on layer 16, net N$4
- removed copper zone on layer 16, net VDD
