File: hw/right.sch (EAGLE design)
At the start: 51 parts, among them J2 CAN, U2 MCP2551, X1 7A-20.000MAAJ-T

Commit message: developing HW version 4.0
Parts:
- C18, C2: value EEE1JA101P -> 100uF
- U$1: device usevolt:MOLEX_MICRO-FIT_10WAY_SMD -> usevolt:MOLEX_MICRO-FIT_10WAY_TH
Changed lines of the file:
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@@
 <part name="P+5" library="supply1" deviceset="+5V" device=""/>
 <part name="GND11" library="supply1" deviceset="GND" device=""/>
-<part name="U$1" library="usevolt" deviceset="MOLEX_MICRO-FIT_10WAY" device="_SMD" value="JOYSTICK"/>
+<part name="U$1" library="usevolt" deviceset="MOLEX_MICRO-FIT_10WAY" device="_TH" value="JOYSTICK"/>
 <part name="F1" library="usevolt" deviceset="FUSE_MC36204_100MA" device="" value="300mA"/>
 <part name="D1" library="usevolt" deviceset="DIODE_TVS_SMBJ33A-TR" device="DO-214AA"/>
@@
 <part name="C1" library="usevolt" deviceset="CAP" device="_0603" value="100n"/>
 <part name="VR1" library="usevolt" deviceset="LM2671" device="SOIC8"/>
-<part name="C2" library="usevolt" deviceset="CAP_POL" device="SMD_10X10X10MM" value="EEE1JA101P"/>
+<part name="C2" library="usevolt" deviceset="CAP_POL" device="SMD_10X10X10MM" value="100uF"/>
 <part name="D23" library="usevolt" deviceset="DIODE" device="DO219AB" value="RS07J-GS18"/>
 <part name="L1" library="usevolt" deviceset="INDUCTOR" device="BOURNS_10X13X5MM" value="SDR1005-101KL"/>
 <part name="C17" library="usevolt" deviceset="CAP" device="_0603" value="10nF"/>
-<part name="C18" library="usevolt" deviceset="CAP_POL" device="SMD_10X10X10MM" value="EEE1JA101P"/>
+<part name="C18" library="usevolt" deviceset="CAP_POL" device="SMD_10X10X10MM" value="100uF"/>
 <part name="D16" library="usevolt" deviceset="DIODE_ZENER" device="SDO123" value="PDZ3.3B,115"/>
 <part name="D17" library="usevolt" deviceset="DIODE_ZENER" device="SDO123" value="PDZ3.3B,115"/>
